File: sswkbd/sswkbd.kicad_pcb (KiCad board)
At the start: 2 copper layers, 160 parts, among them SW1 SW_PUSH, SW10 SW_PUSH, SW11 SW_PUSH, SW12 SW_PUSH, SW13 SW_PUSH, SW14 SW_PUSH, SW15 SW_PUSH, SW16 SW_PUSH, SW17 SW_PUSH, SW18 SW_PUSH, SW19 SW_PUSH, SW2 SW_PUSH, SW20 SW_PUSH, SW21 SW_PUSH, SW22 SW_PUSH, SW23 SW_PUSH, SW24 SW_PUSH, SW25 SW_PUSH, SW26 SW_PUSH, SW27 SW_PUSH, SW28 SW_PUSH, SW29 SW_PUSH, SW3 SW_PUSH, SW30 SW_PUSH, SW31 SW_PUSH, SW32 SW_PUSH, SW33 SW_PUSH, SW34 SW_PUSH, SW35 SW_PUSH, SW36 SW_PUSH, SW37 SW_PUSH, SW38 SW_PUSH, SW39 SW_PUSH, SW4 SW_PUSH, SW40 SW_PUSH, SW41 SW_PUSH, SW42 SW_PUSH, SW43 SW_PUSH, SW44 SW_PUSH, SW45 SW_PUSH, SW46 SW_PUSH, SW47 SW_PUSH, SW48 SW_PUSH, SW49 SW_PUSH, SW5 SW_PUSH, SW50 SW_PUSH, SW51 SW_PUSH, SW52 SW_PUSH, SW53 SW_PUSH, SW54 SW_PUSH, SW55 SW_PUSH, SW56 SW_PUSH, SW57 SW_PUSH, SW58 SW_PUSH, SW59 SW_PUSH, SW6 SW_PUSH, SW60 SW_PUSH, SW61 SW_PUSH, SW62 SW_PUSH, SW63 SW_PUSH, SW64 SW_PUSH, SW65 SW_PUSH, SW66 SW_PUSH, SW67 SW_PUSH, SW68 SW_PUSH, SW69 SW_PUSH, SW7 SW_PUSH, SW70 SW_PUSH, SW71 SW_PUSH, SW72 SW_PUSH, SW73 SW_PUSH, SW74 SW_PUSH, SW75 SW_PUSH, SW76 SW_PUSH, SW77 SW_PUSH, SW78 SW_PUSH, SW79 SW_PUSH, SW8 SW_PUSH, SW9 SW_PUSH, U1 ProMicro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

Commit message: update
Parts:
- added LED1: YS-SK6812MINI-E, kbd:SK6812MINI-E, F.Cu at (33.2, 97.5)
- added LED10: YS-SK6812MINI-E, kbd:SK6812MINI-E, F.Cu at (80.7, 97.5)
- added LED11: YS-SK6812MINI-E, kbd:SK6812MINI-E, F.Cu at (83.1, 116.5)
- added LED12: YS-SK6812MINI-E, kbd:SK6812MINI-E, F.Cu at (87.9, 135.6)
- added LED13: YS-SK6812MINI-E, kbd:SK6812MINI-E, F.Cu at (78.4, 154.6)
- added LED14: YS-SK6812MINI-E, kbd:SK6812MINI-E, F.Cu at (99.8, 154.6)
- added LED15: YS-SK6812MINI-E, kbd:SK6812MINI-E, F.Cu at (118.8, 154.6)
- added LED16: YS-SK6812MINI-E, kbd:SK6812MINI-E, F.Cu at (118.8, 135.6)
- added LED17: YS-SK6812MINI-E, kbd:SK6812MINI-E, F.Cu at (109.3, 116.5)
- added LED18: YS-SK6812MINI-E, kbd:SK6812MINI-E, F.Cu at (104.5, 97.5)
- added LED19: YS-SK6812MINI-E, kbd:SK6812MINI-E, F.Cu at (95.0, 78.4)
- added LED2: YS-SK6812MINI-E, kbd:SK6812MINI-E, F.Cu at (33.2, 116.5)
- added LED20: YS-SK6812MINI-E, kbd:SK6812MINI-E, F.Cu at (114.0, 78.4)
- added LED21: YS-SK6812MINI-E, kbd:SK6812MINI-E, F.Cu at (123.5, 97.5)
- added LED22: YS-SK6812MINI-E, kbd:SK6812MINI-E, F.Cu at (128.3, 116.5)
- added LED23: YS-SK6812MINI-E, kbd:SK6812MINI-E, F.Cu at (137.8, 135.6)
- added LED24: YS-SK6812MINI-E, kbd:SK6812MINI-E, F.Cu at (154.4, 154.6)
- added LED25: YS-SK6812MINI-E, kbd:SK6812MINI-E, F.Cu at (156.8, 135.6)
- added LED26: YS-SK6812MINI-E, kbd:SK6812MINI-E, F.Cu at (142.5, 97.5)
- added LED27: YS-SK6812MINI-E, kbd:SK6812MINI-E, F.Cu at (147.3, 116.5)
- added LED28: YS-SK6812MINI-E, kbd:SK6812MINI-E, F.Cu at (133.0, 78.4)
- added LED29: YS-SK6812MINI-E, kbd:SK6812MINI-E, F.Cu at (152.0, 78.4)
- added LED3: YS-SK6812MINI-E, kbd:SK6812MINI-E, F.Cu at (33.2, 135.6)
- added LED30: YS-SK6812MINI-E, kbd:SK6812MINI-E, F.Cu at (161.5, 97.5)
- added LED31: YS-SK6812MINI-E, kbd:SK6812MINI-E, F.Cu at (166.3, 116.5)
- added LED32: YS-SK6812MINI-E, kbd:SK6812MINI-E, F.Cu at (175.8, 135.6)
- added LED33: YS-SK6812MINI-E, kbd:SK6812MINI-E, F.Cu at (190.0, 154.6)
- added LED34: YS-SK6812MINI-E, kbd:SK6812MINI-E, F.Cu at (194.8, 135.6)
- added LED35: YS-SK6812MINI-E, kbd:SK6812MINI-E, F.Cu at (180.5, 97.5)
- added LED36: YS-SK6812MINI-E, kbd:SK6812MINI-E, F.Cu at (185.3, 116.5)
- added LED37: YS-SK6812MINI-E, kbd:SK6812MINI-E, F.Cu at (171.0, 78.4)
- added LED38: YS-SK6812MINI-E, kbd:SK6812MINI-E, F.Cu at (190.0, 78.4)
- added LED39: YS-SK6812MINI-E, kbd:SK6812MINI-E, F.Cu at (383.4, 97.5)
- added LED4: YS-SK6812MINI-E, kbd:SK6812MINI-E, F.Cu at (33.2, 154.6)
- added LED40: YS-SK6812MINI-E, kbd:SK6812MINI-E, F.Cu at (383.4, 116.5)
- added LED41: YS-SK6812MINI-E, kbd:SK6812MINI-E, F.Cu at (383.4, 135.6)
- added LED42: YS-SK6812MINI-E, kbd:SK6812MINI-E, F.Cu at (383.4, 154.6)
- added LED43: YS-SK6812MINI-E, kbd:SK6812MINI-E, F.Cu at (364.4, 154.6)
- added LED44: YS-SK6812MINI-E, kbd:SK6812MINI-E, F.Cu at (364.4, 135.6)
- added LED45: YS-SK6812MINI-E, kbd:SK6812MINI-E, F.Cu at (352.6, 116.5)
- added LED46: YS-SK6812MINI-E, kbd:SK6812MINI-E, F.Cu at (359.7, 97.5)
- added LED47: YS-SK6812MINI-E, kbd:SK6812MINI-E, F.Cu at (354.9, 78.4)
- added LED48: YS-SK6812MINI-E, kbd:SK6812MINI-E, F.Cu at (326.4, 78.4)
- added LED49: YS-SK6812MINI-E, kbd:SK6812MINI-E, F.Cu at (335.9, 97.5)
- added LED5: YS-SK6812MINI-E, kbd:SK6812MINI-E, F.Cu at (52.2, 154.6)
- added LED50: YS-SK6812MINI-E, kbd:SK6812MINI-E, F.Cu at (338.3, 135.6)
- added LED51: YS-SK6812MINI-E, kbd:SK6812MINI-E, F.Cu at (345.4, 154.6)
- added LED52: YS-SK6812MINI-E, kbd:SK6812MINI-E, F.Cu at (326.4, 154.6)
- added LED53: YS-SK6812MINI-E, kbd:SK6812MINI-E, F.Cu at (307.4, 154.6)
- added LED54: YS-SK6812MINI-E, kbd:SK6812MINI-E, F.Cu at (312.2, 135.6)
- added LED55: YS-SK6812MINI-E, kbd:SK6812MINI-E, F.Cu at (316.9, 97.5)
- added LED56: YS-SK6812MINI-E, kbd:SK6812MINI-E, F.Cu at (321.7, 116.5)
- added LED57: YS-SK6812MINI-E, kbd:SK6812MINI-E, F.Cu at (307.4, 78.4)
- added LED58: YS-SK6812MINI-E, kbd:SK6812MINI-E, F.Cu at (288.4, 78.4)
- added LED59: YS-SK6812MINI-E, kbd:SK6812MINI-E, F.Cu at (297.9, 97.5)
- added LED6: YS-SK6812MINI-E, kbd:SK6812MINI-E, F.Cu at (52.2, 135.6)
- added LED60: YS-SK6812MINI-E, kbd:SK6812MINI-E, F.Cu at (302.7, 116.5)
- added LED61: YS-SK6812MINI-E, kbd:SK6812MINI-E, F.Cu at (293.2, 135.6)
- added LED62: YS-SK6812MINI-E, kbd:SK6812MINI-E, F.Cu at (288.4, 154.6)
- added LED63: YS-SK6812MINI-E, kbd:SK6812MINI-E, F.Cu at (274.2, 135.6)
- added LED64: YS-SK6812MINI-E, kbd:SK6812MINI-E, F.Cu at (283.7, 116.5)
- added LED65: YS-SK6812MINI-E, kbd:SK6812MINI-E, F.Cu at (269.4, 78.4)
- added LED66: YS-SK6812MINI-E, kbd:SK6812MINI-E, F.Cu at (278.9, 97.5)
- added LED67: YS-SK6812MINI-E, kbd:SK6812MINI-E, F.Cu at (250.4, 78.4)
- added LED68: YS-SK6812MINI-E, kbd:SK6812MINI-E, F.Cu at (259.9, 97.5)
- added LED69: YS-SK6812MINI-E, kbd:SK6812MINI-E, F.Cu at (264.7, 116.5)
- added LED7: YS-SK6812MINI-E, kbd:SK6812MINI-E, F.Cu at (52.2, 116.5)
- added LED70: YS-SK6812MINI-E, kbd:SK6812MINI-E, F.Cu at (255.2, 135.6)
- added LED71: YS-SK6812MINI-E, kbd:SK6812MINI-E, F.Cu at (259.9, 154.6)
- added LED72: YS-SK6812MINI-E, kbd:SK6812MINI-E, F.Cu at (245.7, 116.5)
- added LED73: YS-SK6812MINI-E, kbd:SK6812MINI-E, F.Cu at (240.9, 97.5)
- added LED74: YS-SK6812MINI-E, kbd:SK6812MINI-E, F.Cu at (231.4, 78.4)
- added LED75: YS-SK6812MINI-E, kbd:SK6812MINI-E, F.Cu at (221.9, 97.5)
- added LED76: YS-SK6812MINI-E, kbd:SK6812MINI-E, F.Cu at (226.7, 116.5)
- added LED77: YS-SK6812MINI-E, kbd:SK6812MINI-E, F.Cu at (236.2, 135.6)
- added LED78: YS-SK6812MINI-E, kbd:SK6812MINI-E, F.Cu at (231.4, 154.6)
- added LED8: YS-SK6812MINI-E, kbd:SK6812MINI-E, F.Cu at (52.2, 97.5)
- added LED9: YS-SK6812MINI-E, kbd:SK6812MINI-E, F.Cu at (76.0, 78.4)
- moved U2 222.3 mm to (336.7, 216.5)
- moved D56 9.86 mm to (202.9, 133.2)
- moved SW56 9.86 mm to (194.8, 130.8)
- moved D7 9.85 mm to (198.1, 76.1)
- moved D71 9.85 mm to (198.1, 152.3)
- moved SW7 9.85 mm to (190.0, 73.7)
- moved SW71 9.85 mm to (190.0, 149.9)
- moved D40 9.84 mm to (193.4, 114.2)
- moved SW40 9.84 mm to (185.3, 111.8)
- moved D23 9.83 mm to (188.6, 95.1)
- moved SW23 9.83 mm to (180.5, 92.7)
- moved D55 9.81 mm to (183.9, 133.2)
- moved SW55 9.81 mm to (175.8, 130.8)
- moved D6 9.80 mm to (179.1, 76.1)
- moved SW6 9.80 mm to (171.0, 73.7)
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Connections:
- SW15 pad A: (no net) -> unconnected-(SW15-PadA)
- SW15 pad B: (no net) -> unconnected-(SW15-PadB)
- SW15 pad C: (no net) -> GND
- SW15 pad S1: (no net) -> Net-(D15-A)
- SW15 pad S2: Net-(D15-A) -> col_r_0
- U1 pad 20: unconnected-(U1-F4/A3-Pad20) -> col7
Routing:
- net col6: track 0.00 -> 238.7 mm, vias 0 -> 9
- net col7: track 0.00 -> 237.0 mm, vias 0 -> 9
- net col4: track 0.00 -> 203.8 mm, vias 0 -> 11
- net col3: track 0.00 -> 186.0 mm, vias 0 -> 11
- net col5: track 0.00 -> 185.5 mm, vias 0 -> 9
- net row3: track 16.3 -> 177.9 mm
- net row6: track 18.3 -> 179.8 mm
- net col0: track 0.00 -> 158.8 mm, vias 0 -> 3
- net row4: track 14.2 -> 171.1 mm
- net row7: track 16.3 -> 173.0 mm
- net col2: track 0.00 -> 153.7 mm, vias 0 -> 9
- net row2: track 16.3 -> 168.4 mm
- net Net-(D72-K): track 16.3 -> 168.3 mm
- net row1: track 16.3 -> 163.6 mm
- net row8: track 16.3 -> 163.5 mm
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Other:
- board outline added: 3.6 x 3.1 mm

Commit message: PCB WIP
Parts:
- LED1, LED10, LED11, LED12, LED13, LED14, LED15, LED16, LED17, LED18, LED19, LED2, LED20, LED21, LED22, LED23, LED24, LED25, LED26, LED27, LED28, LED29, LED3, LED30, LED31, LED32, LED33, LED34, LED35, LED36, LED37, LED38, LED39, LED4, LED40, LED41, LED42, LED43, LED44, LED45, LED46, LED47, LED48, LED49, LED5, LED50, LED51, LED52, LED53, LED54, LED55, LED56, LED57, LED58, LED59, LED6, LED60, LED61, LED62, LED63, LED64, LED65, LED66, LED67, LED68, LED69, LED7, LED70, LED71, LED72, LED73, LED74, LED75, LED76, LED77, LED78, LED8, LED9: moved to B.Cu
- moved D71 18.4 mm to (179.7, 152.3)
- moved D7 17.1 mm to (181.3, 78.8)
- moved D40 17.0 mm to (176.5, 116.8)
- moved D23 17.0 mm to (171.8, 97.8)
- moved D56 16.9 mm to (186.0, 135.0)
- moved SW15 1.08 mm to (385.3, 72.7)
- moved D65 0.08 mm to (41.3, 152.2)
- moved D66 0.08 mm to (60.3, 152.2)
- moved D67 0.08 mm to (86.5, 152.2)
- moved D68 0.08 mm to (107.9, 152.2)
- moved D69 0.08 mm to (126.9, 152.2)
- moved D70 0.08 mm to (162.5, 152.2)
- moved D72 0.08 mm to (239.5, 152.2)
- moved D73 0.08 mm to (268.0, 152.2)
- moved D74 0.08 mm to (296.5, 152.2)
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Connections:
- LED1 pad 4: unconnected-(LED1-DIN-Pad4) -> LED
- U1 pad 21: unconnected-(U1-VCC-Pad21) -> VCC
- U1 pad 23: unconnected-(U1-GND-Pad23) -> GND
- U1 pad 3: unconnected-(U1-GND-Pad3) -> GND
- U1 pad 4: unconnected-(U1-GND-Pad4) -> GND
- U1 pad 7: unconnected-(U1-4/D4-Pad7) -> LED
Routing:
- net VCC: track 0.00 -> 1100.8 mm, vias 0 -> 64
- net GND: track 0.00 -> 1024.1 mm, vias 0 -> 34
- net row3: track 177.9 -> 14.2 mm
- net row4: track 171.1 -> 12.2 mm
- net row2: track 168.4 -> 14.2 mm
- net row1: track 163.6 -> 14.2 mm
- net row0: track 126.2 -> 10.2 mm
- net Net-(LED5-DOUT): track 0.00 -> 43.2 mm, vias 0 -> 2
- net Net-(LED7-DOUT): track 0.00 -> 34.8 mm, vias 0 -> 2
- net Net-(LED6-DOUT): track 0.00 -> 32.1 mm, vias 0 -> 2
- net Net-(LED4-DOUT): track 0.00 -> 28.2 mm, vias 0 -> 2
- net Net-(LED1-DOUT): track 0.00 -> 20.0 mm, vias 0 -> 2
- net Net-(LED2-DOUT): track 0.00 -> 19.9 mm
- net Net-(LED3-DOUT): track 0.00 -> 19.9 mm
- net LED: track 0.00 -> 18.6 mm, vias 0 -> 1
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Other:
- board size 3.6 x 3.1 mm -> 369.3 x 95.1 mm
