File: sswkbd/sswkbd.kicad_sch (KiCad schematic)
At the start: 238 parts, among them SW1 SW_PUSH, SW10 SW_PUSH, SW11 SW_PUSH, SW12 SW_PUSH, SW13 SW_PUSH, SW14 SW_PUSH, SW15 SW_PUSH, SW16 SW_PUSH, SW17 SW_PUSH, SW18 SW_PUSH, SW19 SW_PUSH, SW2 SW_PUSH, SW20 SW_PUSH, SW21 SW_PUSH, SW22 SW_PUSH, SW23 SW_PUSH, SW24 SW_PUSH, SW25 SW_PUSH, SW26 SW_PUSH, SW27 SW_PUSH, SW28 SW_PUSH, SW29 SW_PUSH, SW3 SW_PUSH, SW30 SW_PUSH, SW31 SW_PUSH, SW32 SW_PUSH, SW33 SW_PUSH, SW34 SW_PUSH, SW35 SW_PUSH, SW36 SW_PUSH, SW37 SW_PUSH, SW38 SW_PUSH, SW39 SW_PUSH, SW4 SW_PUSH, SW40 SW_PUSH, SW41 SW_PUSH, SW42 SW_PUSH, SW43 SW_PUSH, SW44 SW_PUSH, SW45 SW_PUSH, SW46 SW_PUSH, SW47 SW_PUSH, SW48 SW_PUSH, SW49 SW_PUSH, SW5 SW_PUSH, SW50 SW_PUSH, SW51 SW_PUSH, SW52 SW_PUSH, SW53 SW_PUSH, SW54 SW_PUSH, SW55 SW_PUSH, SW56 SW_PUSH, SW57 SW_PUSH, SW58 SW_PUSH, SW59 SW_PUSH, SW6 SW_PUSH, SW60 SW_PUSH, SW61 SW_PUSH, SW62 SW_PUSH, SW63 SW_PUSH, SW64 SW_PUSH, SW65 SW_PUSH, SW66 SW_PUSH, SW67 SW_PUSH, SW68 SW_PUSH, SW69 SW_PUSH, SW7 SW_PUSH, SW70 SW_PUSH, SW71 SW_PUSH, SW72 SW_PUSH, SW73 SW_PUSH, SW74 SW_PUSH, SW75 SW_PUSH, SW76 SW_PUSH, SW77 SW_PUSH, SW78 SW_PUSH, SW79 SW_PUSH, SW8 SW_PUSH, SW9 SW_PUSH, U1 ProMicro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

Commit message: update
Parts:
- LED1, LED10, LED11, LED12, LED13, LED14, LED15, LED16, LED17, LED18, LED19, LED2, LED20, LED21, LED22, LED23, LED24, LED25, LED26, LED27, LED28, LED29, LED3, LED30, LED31, LED32, LED33, LED34, LED35, LED36, LED37, LED38, LED39, LED4, LED40, LED41, LED42, LED43, LED44, LED45, LED46, LED47, LED48, LED49, LED5, LED50, LED51, LED52, LED53, LED54, LED55, LED56, LED57, LED58, LED59, LED6, LED60, LED61, LED62, LED63, LED64, LED65, LED66, LED67, LED68, LED69, LED7, LED70, LED71, LED72, LED73, LED74, LED75, LED76, LED77, LED78, LED8, LED9: footprint (none) -> kbd:SK6812MINI-E
Connections:
- net col0: now also U1.13 (B6/10); no longer U1.19 (F5/A2)
- net col1: now also U1.14 (B2/16); no longer U1.18 (F6/A1)
- net col2: now also U1.15 (B3/14); no longer U1.17 (F7/A0)
- net col4: now also U1.17 (F7/A0); no longer U1.15 (B3/14)
- net col5: now also U1.18 (F6/A1); no longer U1.14 (B2/16)
- net col6: now also U1.19 (F5/A2); no longer U1.13 (B6/10)
- net col7: now also U1.20 (F4/A3)

Commit message: PCB WIP
Connections:
- net GND: now also U1.23 (GND), U1.3 (GND), U1.4 (GND)
- net VCC: now also U1.21 (VCC)
- net LED: now reaches LED1.4 (DIN)
- net LED: now also U1.7 (4/D4)
Changed lines of the file:
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@@
+		)
+	)
+	(global_label "LED"
+		(shape input)
+		(at 31.75 262.89 180)
+		(fields_autoplaced yes)
+		(effects
+			(font
+				(size 1.27 1.27)
+			)
+			(justify right)
+		)
+		(property "Intersheetrefs" "${INTERSHEET_REFS}"
+			(at 25.3177 262.89 0)
+			(effects
+				(font
+					(size 1.27 1.27)
+				)
+				(justify right)
+				(hide yes)
+			)
+		)
+	)
+	(global_label "GND"
+		(shape input)
+		(at 31.75 255.27 180)
+		(fields_autoplaced yes)
+		(effects
+			(font
+				(size 1.27 1.27)
+			)
+			(justify right)
+		)
+		(property "Intersheetrefs" "${INTERSHEET_REFS}"
+			(at 24.8943 255.27 0)
+			(effects
+				(font
+					(size 1.27 1.27)
+				)
+				(justify right)
+				(hide yes)
+			)
 		)
 	)
@@
 		)
 	)
+	(global_label "GND"
+		(shape input)
+		(at 67.31 250.19 0)
+		(fields_autoplaced yes)
+		(effects
+			(font
+				(size 1.27 1.27)
+			)
+			(justify left)
+		)
+		(property "Intersheetrefs" "${INTERSHEET_REFS}"
+			(at 74.1657 250.19 0)
+			(effects
+				(font
+					(size 1.27 1.27)
+				)
+				(justify left)
+				(hide yes)
+			)
+		)
+	)
 	(global_label "row0"
 		(shape input)
@@
 		)
 	)
+	(global_label "GND"
+		(shape input)
+		(at 31.75 252.73 180)
+		(fields_autoplaced yes)
+		(effects
+			(font
+				(size 1.27 1.27)
+			)
+			(justify right)
+		)
+		(property "Intersheetrefs" "${INTERSHEET_REFS}"
+			(at 24.8943 252.73 0)
+			(effects
+				(font
+					(size 1.27 1.27)
+				)
+				(justify right)
+				(hide yes)
+			)
+		)
+	)
 	(global_label "col7"
 		(shape input)
@@
 		)
 	)
+	(global_label "LED"
+		(shape input)
+		(at 33.02 151.13 90)
+		(fields_autoplaced yes)
+		(effects
+			(font
+				(size 1.27 1.27)
+			)
+			(justify left)
+		)
+		(property "Intersheetrefs" "${INTERSHEET_REFS}"
+			(at 33.02 144.6977 90)
+			(effects
+				(font
+					(size 1.27 1.27)
+				)
+				(justify left)
+				(hide yes)
+			)
+		)
+	)
 	(global_label "col_r_5"
 		(shape input)
@@
 			(effects
 				(font
+					(size 1.27 1.27)
+				)
+				(justify left)
+				(hide yes)
+			)
+		)
+	)
+	(global_label "VCC"
+		(shape input)
+		(at 67.31 255.27 0)
+		(fields_autoplaced yes)
+		(effects
+			(font
+				(size 1.27 1.27)
+			)
+			(justify left)
+		)
+		(property "Intersheetrefs" "${INTERSHEET_REFS}"
+			(at 73.9238 255.27 0)
+			(effects
+				(font

Commit message: PCB WIP
Connections:
- net GND: no longer LED39.3 (VSS), LED40.3 (VSS), LED41.3 (VSS), LED42.3 (VSS), LED43.3 (VSS), LED44.3 (VSS), LED45.3 (VSS), LED46.3 (VSS), LED47.3 (VSS), LED48.3 (VSS), LED49.3 (VSS), LED50.3 (VSS), LED51.3 (VSS), LED52.3 (VSS), LED53.3 (VSS), LED54.3 (VSS), LED55.3 (VSS), LED56.3 (VSS), LED57.3 (VSS), LED58.3 (VSS), LED59.3 (VSS), LED60.3 (VSS), LED61.3 (VSS), LED62.3 (VSS), LED63.3 (VSS), LED64.3 (VSS), LED65.3 (VSS), LED66.3 (VSS), LED67.3 (VSS), LED68.3 (VSS), LED69.3 (VSS), LED70.3 (VSS), LED71.3 (VSS), LED72.3 (VSS), LED73.3 (VSS), LED74.3 (VSS), LED75.3 (VSS), LED76.3 (VSS), LED77.3 (VSS), LED78.3 (VSS), SW15.C
- net VCC: no longer LED39.1 (VDD), LED40.1 (VDD), LED41.1 (VDD), LED42.1 (VDD), LED43.1 (VDD), LED44.1 (VDD), LED45.1 (VDD), LED46.1 (VDD), LED47.1 (VDD), LED48.1 (VDD), LED49.1 (VDD), LED50.1 (VDD), LED51.1 (VDD), LED52.1 (VDD), LED53.1 (VDD), LED54.1 (VDD), LED55.1 (VDD), LED56.1 (VDD), LED57.1 (VDD), LED58.1 (VDD), LED59.1 (VDD), LED60.1 (VDD), LED61.1 (VDD), LED62.1 (VDD), LED63.1 (VDD), LED64.1 (VDD), LED65.1 (VDD), LED66.1 (VDD), LED67.1 (VDD), LED68.1 (VDD), LED69.1 (VDD), LED70.1 (VDD), LED71.1 (VDD), LED72.1 (VDD), LED73.1 (VDD), LED74.1 (VDD), LED75.1 (VDD), LED76.1 (VDD), LED77.1 (VDD), LED78.1 (VDD)
- net col_r_0: now also U2.13 (B6/10)
- net col_r_1: now also U2.14 (B2/16); no longer U2.13 (B6/10)
- net col_r_2: now also U2.15 (B3/14); no longer U2.14 (B2/16)
- net col_r_3: now also U2.16 (B1/15); no longer U2.15 (B3/14)
- net col_r_4: now also U2.17 (F7/A0); no longer U2.16 (B1/15)
- net col_r_5: now also U2.18 (F6/A1); no longer U2.17 (F7/A0)
- net col_r_6: now also U2.19 (F5/A2); no longer U2.18 (F6/A1)
- net col_r_7: now also U2.20 (F4/A3); no longer U2.19 (F5/A2)
- net col_r_8: now also U2.7 (4/D4); no longer U2.20 (F4/A3)
- net row9: now also D72.1 (K), D73.1 (K), D74.1 (K), D75.1 (K), D76.1 (K), D77.1 (K), D78.1 (K), D79.1 (K)
- net VCC2: now reaches U2.21 (VCC)
- net VCC2: now also LED39.1 (VDD), LED40.1 (VDD), LED41.1 (VDD), LED42.1 (VDD), LED43.1 (VDD), LED44.1 (VDD), LED45.1 (VDD), LED46.1 (VDD), LED47.1 (VDD), LED48.1 (VDD), LED49.1 (VDD), LED50.1 (VDD), LED51.1 (VDD), LED52.1 (VDD), LED53.1 (VDD), LED54.1 (VDD), LED55.1 (VDD), LED56.1 (VDD), LED57.1 (VDD), LED58.1 (VDD), LED59.1 (VDD), LED60.1 (VDD), LED61.1 (VDD), LED62.1 (VDD), LED63.1 (VDD), LED64.1 (VDD), LED65.1 (VDD), LED66.1 (VDD), LED67.1 (VDD), LED68.1 (VDD), LED69.1 (VDD), LED70.1 (VDD), LED71.1 (VDD), LED72.1 (VDD), LED73.1 (VDD), LED74.1 (VDD), LED75.1 (VDD), LED76.1 (VDD), LED77.1 (VDD), LED78.1 (VDD)
- net GND2: now reaches U2.23 (GND)
- net GND2: now also LED39.3 (VSS), LED40.3 (VSS), LED41.3 (VSS), LED42.3 (VSS), LED43.3 (VSS), LED44.3 (VSS), LED45.3 (VSS), LED46.3 (VSS), LED47.3 (VSS), LED48.3 (VSS), LED49.3 (VSS), LED50.3 (VSS), LED51.3 (VSS), LED52.3 (VSS), LED53.3 (VSS), LED54.3 (VSS), LED55.3 (VSS), LED56.3 (VSS), LED57.3 (VSS), LED58.3 (VSS), LED59.3 (VSS), LED60.3 (VSS), LED61.3 (VSS), LED62.3 (VSS), LED63.3 (VSS), LED64.3 (VSS), LED65.3 (VSS), LED66.3 (VSS), LED67.3 (VSS), LED68.3 (VSS), LED69.3 (VSS), LED70.3 (VSS), LED71.3 (VSS), LED72.3 (VSS), LED73.3 (VSS), LED74.3 (VSS), LED75.3 (VSS), LED76.3 (VSS), LED77.3 (VSS), LED78.3 (VSS), SW15.C, U2.3 (GND), U2.4 (GND)

Commit message: wiring WIP
Connections:
- net col0: now also U1.15 (B3/14); no longer U1.13 (B6/10)
- net col2: now also U1.13 (B6/10); no longer U1.15 (B3/14)
- net col3: now also U1.12 (9/B5); no longer U1.16 (B1/15)
- net col4: now also U1.11 (8/B4); no longer U1.17 (F7/A0)
- net col5: now also U1.10 (7/E6); no longer U1.18 (F6/A1)
- net col6: now also U1.9 (6/D7); no longer U1.19 (F5/A2)
- net col7: now also U1.8 (5/C6); no longer U1.20 (F4/A3)
- net col_r_0: now also U2.15 (B3/14); no longer U2.13 (B6/10)
- net col_r_2: now also U2.13 (B6/10); no longer U2.15 (B3/14)
- net col_r_3: now also U2.12 (9/B5); no longer U2.16 (B1/15)
- net col_r_4: now also U2.11 (8/B4); no longer U2.17 (F7/A0)
- net col_r_5: now also U2.10 (7/E6); no longer U2.18 (F6/A1)
- net col_r_6: now also U2.9 (6/D7); no longer U2.19 (F5/A2)
- net col_r_7: now also U2.8 (5/C6); no longer U2.20 (F4/A3)
- net row0: now also U1.20 (F4/A3); no longer U1.12 (9/B5)
- net row1: now also U1.19 (F5/A2); no longer U1.11 (8/B4)
- net row2: now also U1.18 (F6/A1); no longer U1.10 (7/E6)
- net row3: now also U1.17 (F7/A0); no longer U1.9 (6/D7)
- net row4: now also U1.16 (B1/15); no longer U1.8 (5/C6)
- net row5: now also U2.20 (F4/A3); no longer U2.12 (9/B5)
- net row6: now also U2.19 (F5/A2); no longer U2.11 (8/B4)
- net row7: now also U2.18 (F6/A1); no longer U2.10 (7/E6)
- net row8: now also U2.17 (F7/A0); no longer U2.9 (6/D7)
- net row9: now also U2.16 (B1/15); no longer U2.8 (5/C6)
- net SPLIT_R: now reaches U2.1 (TX0/D3)
- net LED_R: now reaches U2.2 (RX1/D2)
- net RST_R: now reaches U2.22 (RST)
- net SPLIT_L: now reaches U1.1 (TX0/D3)
- net LED_L: now reaches U1.2 (RX1/D2)
- net LED_L: now also LED1.4 (DIN)
- net RST: now reaches U1.22 (RST)
- net LED renamed col8
- net col8: no longer LED1.4 (DIN)
Other:
- moved on the sheet: U2
